File: pcbs/artemis_board/artemis_board.sch (EAGLE design)
At the start: 277 parts, among them J1 10118192-0001LF, J2 FTSH-105-01-F-DV-007-K-P, Q10 BSS138K, Q11 2N7002K-7, Q12 BSS138K, Q13 2N7002K-7, Q14 BSS138K, Q15 2N7002K-7, Q16 BSS138K, Q17 2N7002K-7, Q18 BSS138K, Q19 2N7002K-7, Q20 BSS138K, Q21 2N7002K-7, Q22 BSS138K, Q23 2N7002K-7, Q24 BSS138K, Q25 2N7002K-7, Q26 BSS138K, Q27 2N7002K-7, Q28 BSS138K, Q29 2N7002K-7, Q30 BSS138K, Q31 2N7002K-7, Q32 BSS138K, Q33 2N7002K-7, Q34 BSS138K, Q35 2N7002K-7, Q36 BSS138K, Q5 2N7002K-7, Q6 BSS138K, Q7 2N7002K-7, Q8 BSS138K, Q9 2N7002K-7, U1 ARTEMIS_MODULESMD, U10 CDBHD140L-G, U11 CDBHD140L-G, U12 MAX9938, U13 TN2106K1-G, U14 CDBHD140L-G, U15 CDBHD140L-G, U16 CDBHD140L-G, U17 MAX9938, U18 TN2106K1-G, U19 CDBHD140L-G, U2 CP2102, U20 CDBHD140L-G, U21 74AXP1T45GWH, U22 TMUX1104DGSR, U23 CDBHD140L-G, U24 CDBHD140L-G, U25 MAX9938, U26 TN2106K1-G, U27 TMUX1104DGSR, U28 TMUX1104DGSR, U29 TPS62120, U3 74AXP1T45GWH, U30 TMUX1108RSVR, U31 CDBHD140L-G, U32 CDBHD140L-G, U33 CDBHD140L-G, U34 TMUX1108RSVR, U35 TMUX1108RSVR, U36 TMUX1108RSVR, U37 TMUX1104DGSR, U4 CDBHD140L-G, U5 CDBHD140L-G, U6 CDBHD140L-G, U7 CDBHD140L-G, U8 MAX9938, U9 TN2106K1-G

Commit message: artemis energy harvesting board ready for ordering
Parts:
- R49: MFR (none) -> yageo; MFR_PN (none) -> RC0402FR-07100KL
Changed lines of the file:
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@@
 <setting verticaltext="up"/>
 </settings>
-<grid distance="0.05" unitdist="inch" unit="inch" style="lines" multiple="1" display="yes" altdistance="0.01" altunitdist="inch" altunit="inch"/>
+<grid distance="0.1" unitdist="inch" unit="inch" style="lines" multiple="1" display="no" altdistance="0.01" altunitdist="inch" altunit="inch"/>
 <layers>
 <layer number="1" name="Top" color="4" fill="1" visible="no" active="no"/>
@@
 </part>
 <part name="GND133" library="supply1" library_urn="urn:adsk.eagle:library:371" deviceset="GND" device=""/>
-<part name="R49" library="rcl" library_urn="urn:adsk.eagle:library:334" deviceset="R-US_" device="R0402" package3d_urn="urn:adsk.eagle:package:23547/3" value="100k"/>
+<part name="R49" library="rcl" library_urn="urn:adsk.eagle:library:334" deviceset="R-US_" device="R0402" package3d_urn="urn:adsk.eagle:package:23547/3" value="100k">
+<spice>
+<pinmapping spiceprefix="R">
+<pinmap gate="G$1" pin="1" pinorder="1"/>
+<pinmap gate="G$1" pin="2" pinorder="2"/>
+</pinmapping>
+</spice>
+<attribute name="MFR" value="yageo"/>
+<attribute name="MFR_PN" value="RC0402FR-07100KL"/>
+</part>
 <part name="P+1" library="supply1" library_urn="urn:adsk.eagle:library:371" deviceset="VCC" device=""/>
 <part name="GND134" library="supply1" library_urn="urn:adsk.eagle:library:371" deviceset="GND" device=""/>
@@
 <attribute name="NAME" x="133.1214" y="-109.22" size="1.778" layer="95" rot="R90"/>
 <attribute name="VALUE" x="137.922" y="-109.22" size="1.778" layer="96" rot="R90"/>
+<attribute name="MFR" x="134.62" y="-105.41" size="1.778" layer="96" rot="R90" display="off"/>
+<attribute name="MFR_PN" x="134.62" y="-105.41" size="1.778" layer="96" rot="R90" display="off"/>
 </instance>
 <instance part="P+1" gate="VCC" x="134.62" y="-96.52" smashed="yes">
