File: pcbs/adaptor_board/afig-adaptor.brd (EAGLE design)
At the start: 9 x 9.1 mm, 2 parts

Commit message: wip
Parts:
- added J1: B2B-PH-SM4-TB, JST-PH:B2B-PH-SM4-TB
- moved U$1 0.76 mm to (0.00, -0.10)
- moved U$2 0.76 mm to (0.00, -0.70)
Connections:
- net N$3: now also J1.P$1
- net N$4: now also J1.P$2
Routing:
- net N$4: track 4.09 -> 8.72 mm, vias 0 -> 1
- net N$3: track 4.59 -> 7.87 mm
- net N$1: track 9.62 -> 10.7 mm
Other:
- board size 9 x 9.1 mm -> 9.4 x 9.4 mm
