File: pcbs/adaptor_board/afig-adaptor.sch (EAGLE design)
At the start: 2 parts

Commit message: wip
Parts:
- added J1: B2B-PH-SM4-TB, JST-PH:B2B-PH-SM4-TB
Connections:
- net N$3: now also J1.P$1
- net N$4: now also J1.P$2
