File: pcbs/coil_harvester_board/coil_havester_board.brd (EAGLE design)
At the start: 25 x 26 mm, 23 parts, among them U1 CDBHD140L-G, U2 CDBHD140L-G, U3 MAX9938, U4 TN2106K1-G

Commit message: wip
Other:
- board text added: "dirsense"
- board text added: "gnd"
- board text added: "isense"
- board text added: "vharvest"
- board text added: "vrectified"
- board text added: "vsense"
Changed lines of the file:
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@@
 <text x="19.1" y="21.2" size="1" layer="21">Sense</text>
 <text x="18.6" y="12.2" size="1" layer="21">Harvest</text>
+<text x="24.1" y="19" size="0.8" layer="22" rot="MR0" align="center-left">dirsense</text>
+<text x="24.1" y="18" size="0.8" layer="22" rot="MR0" align="center-left">vsense</text>
+<text x="24.1" y="17" size="0.8" layer="22" rot="MR0" align="center-left">isense</text>
+<text x="24.1" y="16" size="0.8" layer="22" rot="MR0" align="center-left">gnd</text>
+<text x="24.1" y="9" size="0.8" layer="22" rot="MR0" align="center-left">vharvest</text>
+<text x="24.1" y="10" size="0.8" layer="22" rot="MR0" align="center-left">vrectified</text>
+<text x="24.1" y="8" size="0.8" layer="22" rot="MR0" align="center-left">gnd</text>
+<text x="24.1" y="7" size="0.8" layer="22" rot="MR0" align="center-left">gnd</text>
 </plain>
 <attributes>
@@
 <attribute name="MFR" value="YAGEO" x="10.2" y="24.1" size="1.778" layer="27" rot="R270" display="off"/>
 <attribute name="MFR_PN" value="RC0402FR-071ML" x="10.2" y="24.1" size="1.778" layer="27" rot="R270" display="off"/>
-<attribute name="NAME" x="12.835" y="24.735" size="0.7" layer="25" rot="R270"/>
+<attribute name="NAME" x="12.7" y="23.5" size="0.7" layer="25" rot="R90"/>
 <attribute name="POPULARITY" value="34" x="10.2" y="24.1" size="1.778" layer="27" rot="R270" display="off"/>
 <attribute name="SPICEPREFIX" value="R" x="10.2" y="24.1" size="1.778" layer="27" rot="R270" display="off"/>
@@
 <attribute name="MFR" value="YAGEO" x="11.3" y="24.1" size="1.778" layer="27" rot="R90" display="off"/>
 <attribute name="MFR_PN" value="RC0402FR-07150KL" x="11.3" y="24.1" size="1.778" layer="27" rot="R90" display="off"/>
-<attribute name="NAME" x="12.565" y="23.465" size="0.7" layer="25" rot="R90"/>
+<attribute name="NAME" x="13.6" y="23.5" size="0.7" layer="25" rot="R90"/>
 <attribute name="POPULARITY" value="34" x="11.3" y="24.1" size="1.778" layer="27" rot="R90" display="off"/>
 <attribute name="SPICEPREFIX" value="R" x="11.3" y="24.1" size="1.778" layer="27" rot="R90" display="off"/>
@@
 <attribute name="MFR" value="JST" x="22" y="8.5" size="1.778" layer="27" rot="R90" display="off"/>
 <attribute name="MFR_PN" value="SM04B-SRSS-TB(LF)(SN)" x="22" y="8.5" size="1.778" layer="27" rot="R90" display="off"/>
-<attribute name="NAME" x="22.505" y="7.83" size="0.3048" layer="25" rot="R90"/>
-<attribute name="VALUE" x="23" y="7.83" size="0.3048" layer="27" rot="R90"/>
 </element>
 <element name="JP3" library="jst-sh" package="JST-SH-4" value="JST-SH-4" x="22" y="17.5" smashed="yes" rot="R90">
 <attribute name="MFR" value="JST" x="22" y="17.5" size="1.778" layer="27" rot="R90" display="off"/>
 <attribute name="MFR_PN" value="SM04B-SRSS-TB(LF)(SN)" x="22" y="17.5" size="1.778" layer="27" rot="R90" display="off"/>
-<attribute name="NAME" x="22.505" y="16.83" size="0.3048" layer="25" rot="R90"/>
-<attribute name="VALUE" x="23" y="16.83" size="0.3048" layer="27" rot="R90"/>
 </element>
 <element name="D1" library="SparkFun-DiscreteSemi" library_urn="urn:adsk.eagle:library:514" package="SOD-323" package3d_urn="urn:adsk.eagle:package:38441/1" value="3.3V" x="15.6" y="1.7" smashed="yes" rot="R180">
@@
 <via x="11.3" y="5.5" extent="1-16" drill="0.35"/>
 <contactref element="JP2" pad="1"/>
-<via x="17.4" y="17.7" extent="1-16" drill="0.35"/>
+<via x="18.2" y="17.8" extent="1-16" drill="0.35"/>
 <via x="14.9" y="2.8" extent="1-16" drill="0.35"/>
 <contactref element="JP2" pad="2"/>
@@
 <wire x1="18.05" y1="1.7" x2="18.15" y2="1.6" width="0.1524" layer="1"/>
 <contactref element="JP2" pad="3"/>
-<wire x1="19.66" y1="9" x2="20.8" y2="9" width="0.3048" layer="1"/>
 <wire x1="20.8" y1="9" x2="21.1" y2="8.7" width="0.3048" layer="1"/>
 <wire x1="21.1" y1="8.7" x2="21.1" y2="5.7" width="0.3048" layer="1"/>
@@
 <wire x1="20.6" y1="5.2" x2="18.2" y2="5.2" width="0.3048" layer="1"/>
 <wire x1="17.9" y1="4.6" x2="17.5" y2="4.2" width="0.3048" layer="1"/>
+<wire x1="19.66" y1="9" x2="20.8" y2="9" width="0.1524" layer="1"/>
 </signal>
 <signal name="N$6">
@@
 <wire x1="20.5" y1="3.8" x2="21.8" y2="5.1" width="0.3048" layer="1"/>
 <wire x1="21.8" y1="5.1" x2="21.8" y2="9.4" width="0.3048" layer="1"/>
-<wire x1="21.8" y1="9.4" x2="21.2" y2="10" width="0.3048" layer="1"/>
-<wire x1="21.2" y1="10" x2="19.66" y2="10" width="0.3048" layer="1"/>
+<wire x1="21.2" y1="10" x2="21.8" y2="9.4" width="0.3048" layer="1"/>
+<wire x1="19.66" y1="10" x2="21.2" y2="10" width="0.1524" layer="1"/>
 </signal>
 </signals>
